Commit message: diffbotの設定内容をSANEHAL向けに修正

File: sanehal_vehicle_description/urdf/diffbot_description.urdf.xacro (robot description, xacro)
@@ -4,14 +4,16 @@
   <!-- Constants for robot dimensions -->
   <xacro:property name="PI" value="3.1415926535897931"/>
-  <xacro:property name="base_mass" value="0.3" /> <!-- arbitrary value for base mass -->
-  <xacro:property name="base_width" value="0.268" />
-  <xacro:property name="base_length" value="0.268" />
-  <xacro:property name="base_height" value="0.05" />
-  <xacro:property name="wheel_mass" value="0.3" /> <!-- arbitrary value for wheel mass -->
+  <xacro:property name="base_mass" value="2.0" /> <!-- arbitrary value for base mass -->
+  <xacro:property name="base_width" value="0.30750" /><!-- x -->
+  <xacro:property name="base_length" value="0.268" /><!-- y -->
+  <xacro:property name="base_height" value="0.45542" /> <!-- z -->
+  <xacro:property name="wheel_mass" value="0.100" /> <!-- arbitrary value for wheel mass -->
   <xacro:property name="wheel_len" value="0.020" />
-  <xacro:property name="wheel_radius" value="0.0395" /> <!-- = 0.079/2 -->
-  <xacro:property name="caster_wheel_mass" value="0.1" /> <!-- arbitrary value for caster wheel mass -->
-  <xacro:property name="caster_wheel_radius" value="0.015" />
-  <xacro:property name="z_offset" value="-${base_height/2}" /> <!-- Space btw top of beam and the each joint -->
+  <xacro:property name="wheel_radius" value="0.03925" /> <!-- = 0.0785/2 -->
+  <xacro:property name="wheel_x_offset" value="0.12525" />
+  <xacro:property name="caster_wheel_mass" value="0.03" /> <!-- arbitrary value for caster wheel mass -->
+  <xacro:property name="caster_wheel_x_offset" value="-0.09175" /> <!-- arbitrary value for caster wheel mass -->
+  <xacro:property name="caster_wheel_radius" value="0.020" />
+  <xacro:property name="z_offset" value="-0" /> <!-- Space btw top of beam and the each joint -->
   <!-- <link name="dummy"></link>
   <joint name="dummy_joint" type="fixed">
@@ -32,5 +34,5 @@
         <box size="${base_width} ${base_length} ${base_height}"/>
       </geometry>
-      <material name="orange"/>
+      <material name="blue"/>
     </visual>
     <inertial>
@@ -46,5 +48,5 @@
       <parent link="${prefix}base_link"/>
       <child link="${prefix}left_wheel"/>
-      <origin xyz="0 -${base_width/2} ${z_offset}" rpy="0 0 0"/>
+      <origin xyz="${wheel_x_offset} ${base_width/2} ${z_offset}" rpy="0 0 0"/>
       <axis xyz="0 1 0"/>
       <dynamics damping="0.2"/>
@@ -77,5 +79,5 @@
       <parent link="${prefix}base_link"/>
       <child link="${prefix}right_wheel"/>
-      <origin xyz="0 ${base_width/2} ${z_offset}" rpy="0 0 0"/>
+      <origin xyz="${wheel_x_offset} -${base_width/2} ${z_offset}" rpy="0 0 ${PI}"/>
       <axis xyz="0 1 0"/>
       <dynamics damping="0.2"/>
@@ -94,5 +96,5 @@
           <cylinder length="${wheel_len}" radius="${wheel_radius}"/>
         </geometry>
-        <material name="black"/>
+        <material name="grey"/>
       </visual>
       <inertial>
@@ -103,33 +105,4 @@
           iyy="${wheel_mass / 12.0 * wheel_radius*wheel_radius}" iyz="0.0"
           izz="${wheel_mass / 12.0 * wheel_radius*wheel_radius}"/>
-        </inertial>
-      </link>
-    <joint name="${prefix}caster_frontal_wheel_joint" type="fixed">
-      <parent link="${prefix}base_link"/>
-      <child link="${prefix}caster_frontal_wheel"/>
-      <origin xyz="${base_width/2 - caster_wheel_radius} 0 ${z_offset}" rpy="0 0 0"/>
-    </joint>
-    <!-- caster frontal wheel Link -->
-    <link name="${prefix}caster_frontal_wheel">
-      <collision>
-        <origin xyz="0 0 0" rpy="0 0 0"/>
-        <geometry>
-          <sphere radius="${caster_wheel_radius}"/>
-        </geometry>
-      </collision>
-      <visual>
-        <origin xyz="0 0 0" rpy="0 0 0"/>
-        <geometry>
-          <sphere radius="${caster_wheel_radius}"/>
-        </geometry>
-        <material name="white"/>
-      </visual>
-      <inertial>
-        <origin xyz="0 0 0" rpy="0 0 0"/>
-        <mass value="${caster_wheel_mass}"/>
-        <inertia
-          ixx="${caster_wheel_mass * 0.4 * (caster_wheel_radius * caster_wheel_radius)}" ixy="0.0" ixz="0.0"
-          iyy="${caster_wheel_mass * 0.4 * (caster_wheel_radius * caster_wheel_radius)}" iyz="0.0"
-          izz="${caster_wheel_mass * 0.4 * (caster_wheel_radius * caster_wheel_radius)}"/>
         </inertial>
       </link>

Commit message: temp commit

File: sanehal_vehicle_description/urdf/diffbot_description.urdf.xacro (robot description, xacro)
@@ -1,4 +1,5 @@
 <?xml version="1.0"?>
 <robot xmlns:xacro="http://www.ros.org/wiki/xacro">
+<!-- ロボットの表示を行う本体部分 -->
   <xacro:macro name="diffbot" params="prefix">
   <!-- Constants for robot dimensions -->
@@ -16,9 +17,4 @@
   <xacro:property name="caster_wheel_radius" value="0.020" />
   <xacro:property name="z_offset" value="-0" /> <!-- Space btw top of beam and the each joint -->
-  <!-- <link name="dummy"></link>
-  <joint name="dummy_joint" type="fixed">
-    <parent link="dummy"/>
-    <child link="${prefix}base_link"/>
-  </joint> -->
   <!-- Base Link -->
   <link name="${prefix}base_link">
