Commit message: temp_update

File: sanehal_vehicle_description/urdf/diffbot.urdf.xacro (robot description, xacro)
@@ -3,5 +3,5 @@
 <robot xmlns:xacro="http://www.ros.org/wiki/xacro" name="diffdrive_robot">
   <xacro:arg name="prefix" default="" />
-  <xacro:include filename="$(find sanehal_vehicle_description)/urdf/diffbot_description.urdf.xacro" />
+  <xacro:include filename="$(find sanehal_vehicle_description)/urdf/diffbot.xacro" />
   <!-- Import Rviz colors -->
   <xacro:include filename="$(find sanehal_vehicle_description)/gazebo/diffbot.materials.xacro" />

File: sanehal_vehicle_description/urdf/diffbot.xacro (robot description, xacro)
@@ -1,5 +1,5 @@
-<?xml version="1.0"?>
+<?xml version="1.0" encoding="UTF-8"?>
 <robot xmlns:xacro="http://www.ros.org/wiki/xacro">
-<!-- ロボットの表示を行う本体部分 -->
+  <!-- ロボットの表示を行う本体部分 -->
   <xacro:macro name="diffbot" params="prefix">
   <!-- Constants for robot dimensions -->
@@ -17,35 +17,36 @@
   <xacro:property name="caster_wheel_radius" value="0.020" />
   <xacro:property name="z_offset" value="-0" /> <!-- Space btw top of beam and the each joint -->
-  <!-- Base Link -->
-  <link name="${prefix}base_link">
-    <collision>
-      <origin xyz="0 0 0" rpy="0 0 0"/>
-      <geometry>
-        <box size="${base_width} ${base_length} ${base_height}"/>
-      </geometry>
-    </collision>
-    <visual>
-      <origin xyz="0 0 ${base_height/2}" rpy="0 0 0"/>
-      <geometry>
-        <box size="${base_width} ${base_length} ${base_height}"/>
-      </geometry>
-      <material name="blue"/>
-    </visual>
-    <inertial>
-      <origin xyz="0 0 0" rpy="0 0 0"/>
-      <mass value="${base_mass}"/>
-      <inertia
-        ixx="${base_mass / 12.0 * (base_length*base_length + base_height*base_height)}" ixy="0.0" ixz="0.0"
-        iyy="${base_mass / 12.0 * (base_height*base_height + base_width*base_width)}" iyz="0.0"
-        izz="${base_mass / 12.0 * (base_width*base_width + base_length*base_length)}"/>
-      </inertial>
+  <!-- <xacro:include filename="$(find ldlidar_stl_description)/urdf/ld19.xacro" /> -->
+    <!-- Base Link -->
+    <link name="${prefix}base_link">
+      <collision>
+        <origin xyz="0 0 0" rpy="0 0 0"/>
+        <geometry>
+          <box size="${base_width} ${base_length} ${base_height}"/>
+        </geometry>
+      </collision>
+      <visual>
+        <origin xyz="0 0 ${base_height/2}" rpy="0 0 0"/>
+        <geometry>
+          <box size="${base_width} ${base_length} ${base_height}"/>
+        </geometry>
+        <material name="blue"/>
+      </visual>
+      <inertial>
+        <origin xyz="0 0 0" rpy="0 0 0"/>
+        <mass value="${base_mass}"/>
+        <inertia
+          ixx="${base_mass / 12.0 * (base_length*base_length + base_height*base_height)}" ixy="0.0" ixz="0.0"
+          iyy="${base_mass / 12.0 * (base_height*base_height + base_width*base_width)}" iyz="0.0"
+          izz="${base_mass / 12.0 * (base_width*base_width + base_length*base_length)}"/>
+        </inertial>
     </link>
-    <joint name="${prefix}left_wheel_joint" type="continuous">
-      <parent link="${prefix}base_link"/>
-      <child link="${prefix}left_wheel"/>
-      <origin xyz="${wheel_x_offset} ${base_width/2} ${z_offset}" rpy="0 0 0"/>
-      <axis xyz="0 1 0"/>
-      <dynamics damping="0.2"/>
-    </joint>
+    <!-- Lidar sensor-->
+    <!-- <xacro:ld19
+      parent="${prefix}base_link"
+      prefix="${prefix}"
+      sensor_range_visible="false">
+      <origin xyz="0 0 0" rpy="0 0 0" />
+    </xacro:ld19> -->
     <!-- left wheel Link -->
     <link name="${prefix}left_wheel">
@@ -71,12 +72,5 @@
           izz="${wheel_mass / 12.0 * wheel_radius*wheel_radius}"/>
         </inertial>
-      </link>
-    <joint name="${prefix}right_wheel_joint" type="continuous">
-      <parent link="${prefix}base_link"/>
-      <child link="${prefix}right_wheel"/>
-      <origin xyz="${wheel_x_offset} -${base_width/2} ${z_offset}" rpy="0 0 ${PI}"/>
-      <axis xyz="0 1 0"/>
-      <dynamics damping="0.2"/>
-    </joint>
+    </link>
     <!-- right wheel Link -->
     <link name="${prefix}right_wheel">
@@ -102,10 +96,5 @@
           izz="${wheel_mass / 12.0 * wheel_radius*wheel_radius}"/>
         </inertial>
-      </link>
-    <joint name="${prefix}caster_rear_wheel_joint" type="fixed">
-      <parent link="${prefix}base_link"/>
-      <child link="${prefix}caster_rear_wheel"/>
-      <origin xyz="${-base_width/2 + caster_wheel_radius} 0 ${z_offset}" rpy="0 0 0"/>
-    </joint>
+    </link>
     <!-- caster rear wheel Link -->
     <link name="${prefix}caster_rear_wheel">
@@ -131,5 +120,25 @@
           izz="${caster_wheel_mass * 0.4 * (caster_wheel_radius * caster_wheel_radius)}"/>
         </inertial>
-      </link>
+    </link>
+    <!-- joints -->
+    <joint name="${prefix}left_wheel_joint" type="continuous">
+      <parent link="${prefix}base_link"/>
+      <child link="${prefix}left_wheel"/>
+      <origin xyz="${wheel_x_offset} ${base_width/2} ${z_offset}" rpy="0 0 0"/>
+      <axis xyz="0 1 0"/>
+      <dynamics damping="0.2"/>
+    </joint>
+    <joint name="${prefix}right_wheel_joint" type="continuous">
+      <parent link="${prefix}base_link"/>
+      <child link="${prefix}right_wheel"/>
+      <origin xyz="${wheel_x_offset} -${base_width/2} ${z_offset}" rpy="0 0 ${PI}"/>
+      <axis xyz="0 1 0"/>
+      <dynamics damping="0.2"/>
+    </joint>
+    <joint name="${prefix}caster_rear_wheel_joint" type="f">
+      <parent link="${prefix}base_link"/>
+      <child link="${prefix}caster_rear_wheel"/>
+      <origin xyz="${-base_width/2 + caster_wheel_radius} 0 ${z_offset}" rpy="0 0 0"/>
+    </joint>
   </xacro:macro>
 </robot>
