Commit message: tempcommit

File: sanehal_vehicle_description/urdf/diffbot.xacro (robot description, xacro)
@@ -1,21 +1,22 @@
 <?xml version="1.0" encoding="UTF-8"?>
-<robot xmlns:xacro="http://www.ros.org/wiki/xacro">
-  <!-- ロボットの表示を行う本体部分 -->
-  <xacro:macro name="diffbot" params="prefix">
-  <!-- Constants for robot dimensions -->
-  <xacro:property name="PI" value="3.1415926535897931"/>
-  <xacro:property name="base_mass" value="2.0" /> <!-- arbitrary value for base mass -->
-  <xacro:property name="base_width" value="0.30750" /><!-- x -->
-  <xacro:property name="base_length" value="0.268" /><!-- y -->
-  <xacro:property name="base_height" value="0.45542" /> <!-- z -->
-  <xacro:property name="wheel_mass" value="0.100" /> <!-- arbitrary value for wheel mass -->
-  <xacro:property name="wheel_len" value="0.020" />
-  <xacro:property name="wheel_radius" value="0.03925" /> <!-- = 0.0785/2 -->
-  <xacro:property name="wheel_x_offset" value="0.12525" />
-  <xacro:property name="caster_wheel_mass" value="0.03" /> <!-- arbitrary value for caster wheel mass -->
-  <xacro:property name="caster_wheel_x_offset" value="-0.09175" /> <!-- arbitrary value for caster wheel mass -->
-  <xacro:property name="caster_wheel_radius" value="0.020" />
-  <xacro:property name="z_offset" value="-0" /> <!-- Space btw top of beam and the each joint -->
-  <!-- <xacro:include filename="$(find ldlidar_stl_description)/urdf/ld19.xacro" /> -->
+  <robot xmlns:xacro="http://www.ros.org/wiki/xacro">
+    <!-- ロボットの表示を行う本体部分 -->
+    <xacro:macro name="diffbot" params="prefix parent">
+    <!-- Constants for robot dimensions -->
+    <xacro:property name="PI" value="3.1415926535897931"/>
+    <xacro:property name="base_mass" value="2.0" /> <!-- arbitrary value for base mass -->
+    <xacro:property name="base_width" value="0.30750" /><!-- x -->
+    <xacro:property name="base_length" value="0.268" /><!-- y -->
+    <xacro:property name="base_height" value="0.45542" /> <!-- z -->
+    <xacro:property name="wheel_mass" value="0.100" /> <!-- arbitrary value for wheel mass -->
+    <xacro:property name="wheel_len" value="0.020" />
+    <xacro:property name="wheel_radius" value="0.03925" /> <!-- = 0.0785/2 -->
+    <xacro:property name="wheel_x_offset" value="0.12525" />
+    <xacro:property name="caster_wheel_mass" value="0.03" /> <!-- arbitrary value for caster wheel mass -->
+    <xacro:property name="caster_wheel_x_offset" value="-0.09175" /> <!-- arbitrary value for caster wheel mass -->
+    <xacro:property name="caster_wheel_radius" value="0.020" />
+    <xacro:property name="z_offset" value="-0" /> <!-- Space btw top of beam and the each joint -->
+    <!-- add sensor file  -->
+    <xacro:include filename="$(find ldlidar_stl_description)/urdf/ld19.xacro" />
     <!-- Base Link -->
     <link name="${prefix}base_link">
@@ -43,10 +44,10 @@
     </link>
     <!-- Lidar sensor-->
-    <!-- <xacro:ld19
+    <xacro:ld19
       parent="${prefix}base_link"
       prefix="${prefix}"
       sensor_range_visible="false">
       <origin xyz="0 0 0" rpy="0 0 0" />
-    </xacro:ld19> -->
+    </xacro:ld19>
     <!-- left wheel Link -->
     <link name="${prefix}left_wheel">
@@ -122,4 +123,5 @@
     </link>
     <!-- joints -->
+    <joint
     <joint name="${prefix}left_wheel_joint" type="continuous">
       <parent link="${prefix}base_link"/>
@@ -136,5 +138,5 @@
       <dynamics damping="0.2"/>
     </joint>
-    <joint name="${prefix}caster_rear_wheel_joint" type="f">
+    <joint name="${prefix}caster_rear_wheel_joint" type="fixed">
       <parent link="${prefix}base_link"/>
       <child link="${prefix}caster_rear_wheel"/>

Commit message: temp

File: sanehal_vehicle_description/urdf/diffbot.xacro (robot description, xacro)
@@ -2,5 +2,5 @@
   <robot xmlns:xacro="http://www.ros.org/wiki/xacro">
     <!-- ロボットの表示を行う本体部分 -->
-    <xacro:macro name="diffbot" params="prefix parent">
+    <xacro:macro name="diffbot" params="prefix parent *origin">
     <!-- Constants for robot dimensions -->
     <xacro:property name="PI" value="3.1415926535897931"/>
@@ -20,5 +20,5 @@
     <xacro:include filename="$(find ldlidar_stl_description)/urdf/ld19.xacro" />
     <!-- Base Link -->
-    <link name="${prefix}base_link">
+    <link name="${prefix}sanehal_base_link">
       <collision>
         <origin xyz="0 0 0" rpy="0 0 0"/>
@@ -45,5 +45,5 @@
     <!-- Lidar sensor-->
     <xacro:ld19
-      parent="${prefix}base_link"
+      parent="${prefix}sanehal_base_link"
       prefix="${prefix}"
       sensor_range_visible="false">
@@ -124,6 +124,12 @@
     <!-- joints -->
     <joint
+        name="${prefix}base_joint"
+        type="fixed">
+      <parent link="${parent}" />
+      <child link="${prefix}sanehal_base_link" />
+      <xacro:insert_block name="origin" />
+    </joint>
     <joint name="${prefix}left_wheel_joint" type="continuous">
-      <parent link="${prefix}base_link"/>
+      <parent link="${prefix}sanehal_base_link"/>
       <child link="${prefix}left_wheel"/>
       <origin xyz="${wheel_x_offset} ${base_width/2} ${z_offset}" rpy="0 0 0"/>
@@ -132,5 +138,5 @@
     </joint>
     <joint name="${prefix}right_wheel_joint" type="continuous">
-      <parent link="${prefix}base_link"/>
+      <parent link="${prefix}sanehal_base_link"/>
       <child link="${prefix}right_wheel"/>
       <origin xyz="${wheel_x_offset} -${base_width/2} ${z_offset}" rpy="0 0 ${PI}"/>
@@ -139,5 +145,5 @@
     </joint>
     <joint name="${prefix}caster_rear_wheel_joint" type="fixed">
-      <parent link="${prefix}base_link"/>
+      <parent link="${prefix}sanehal_base_link"/>
       <child link="${prefix}caster_rear_wheel"/>
       <origin xyz="${-base_width/2 + caster_wheel_radius} 0 ${z_offset}" rpy="0 0 0"/>

File: sanehal_vehicle_description/urdf/diffbot_display.urdf.xacro (robot description, xacro)
@@ -3,9 +3,7 @@
 <robot xmlns:xacro="http://www.ros.org/wiki/xacro" name="diffdrive_robot">
   <xacro:arg name="prefix" default="" />
-  <xacro:include filename="$(find sanehal_vehicle_description)/urdf/diffbot.xacro" />
   <!-- Import Rviz colors -->
   <xacro:include filename="$(find sanehal_vehicle_description)/gazebo/diffbot.materials.xacro" />
-  <!-- Import diffbot ros2_control description -->
-  <xacro:include filename="$(find sanehal_vehicle_description)/ros2_control/diffbot.ros2_control.xacro" />
+  <xacro:include filename="$(find sanehal_vehicle_description)/urdf/diffbot.xacro" />
   <link name="$(arg prefix)base_link" />
   <xacro:diffbot
@@ -16,5 +14,3 @@
         rpy="0 0 0" />
   </xacro:diffbot>
-  <xacro:diffbot_ros2_control
-    name="Sanehal" prefix="$(arg prefix)" />
 </robot>
