Commit message: Add JT16 frame to SANEHAL-2 description

File: sanehal_vehicle_description/urdf/sanehal.urdf.xacro (robot description, xacro)
@@ -3,4 +3,7 @@
 <robot xmlns:xacro="http://www.ros.org/wiki/xacro" name="diffdrive_robot">
   <xacro:arg name="prefix" default="" />
+  <xacro:arg name="jt16_link_name" default="lidar_link" />
+  <xacro:arg name="jt16_xyz" default="0 0 0" />
+  <xacro:arg name="jt16_rpy" default="0 0 0" />
   <xacro:include filename="$(find sanehal_vehicle_description)/urdf/sanehal.xacro" />
   <!-- Import Rviz colors -->
@@ -11,4 +14,7 @@
   <xacro:sanehal
       prefix="$(arg prefix)"
+      jt16_link_name="$(arg jt16_link_name)"
+      jt16_xyz="$(arg jt16_xyz)"
+      jt16_rpy="$(arg jt16_rpy)"
       parent="$(arg prefix)base_link">
     <origin

File: sanehal_vehicle_description/urdf/sanehal.xacro (robot description, xacro)
@@ -2,5 +2,5 @@
   <robot xmlns:xacro="http://www.ros.org/wiki/xacro">
     <!-- ロボットの表示を行う本体部分 -->
-    <xacro:macro name="sanehal" params="prefix parent *origin">
+    <xacro:macro name="sanehal" params="prefix parent jt16_link_name:=lidar_link jt16_xyz:='0 0 0' jt16_rpy:='0 0 0' *origin">
     <!-- Constants for robot dimensions -->
     <xacro:property name="PI" value="3.1415926535897931"/>
@@ -22,6 +22,4 @@
     <xacro:property name="caster_wheel_z_offset" value="0.0124" />
     <xacro:property name="caster_wheel_radius" value="0.0124" />
-    <!-- add sensor file  -->
-    <xacro:include filename="$(find ldlidar_stl_description)/urdf/ld19.xacro" />
     <!-- Base Link -->
     <link name="${prefix}sanehal_base_link">
@@ -48,11 +46,13 @@
         </inertial>
     </link>
-    <!-- Lidar sensor-->
-    <xacro:ld19
-      parent="${prefix}sanehal_base_link"
-      prefix="${prefix}"
-      sensor_range_visible="false">
-      <origin xyz="0 0 0" rpy="0 0 0" />
-    </xacro:ld19>
+    <!-- JT16 sensor frame.
+         Geometry is intentionally omitted until a vendor mesh or measured size is provided.
+         The frame exists so Issue #30 can reuse the same TF frame_id. -->
+    <link name="${prefix}${jt16_link_name}" />
+    <joint name="${prefix}jt16_joint" type="fixed">
+      <parent link="${prefix}sanehal_base_link" />
+      <child link="${prefix}${jt16_link_name}" />
+      <origin xyz="${jt16_xyz}" rpy="${jt16_rpy}" />
+    </joint>
     <!-- left wheel Link -->
     <link name="${prefix}left_wheel">

File: sanehal_vehicle_description/urdf/sanehal_display.urdf.xacro (robot description, xacro)
@@ -3,4 +3,7 @@
 <robot xmlns:xacro="http://www.ros.org/wiki/xacro" name="diffdrive_robot">
   <xacro:arg name="prefix" default="" />
+  <xacro:arg name="jt16_link_name" default="lidar_link" />
+  <xacro:arg name="jt16_xyz" default="0 0 0" />
+  <xacro:arg name="jt16_rpy" default="0 0 0" />
   <!-- Import Rviz colors -->
   <xacro:include filename="$(find sanehal_vehicle_description)/gazebo/sanehal.materials.xacro" />
@@ -9,4 +12,7 @@
   <xacro:sanehal
       prefix="$(arg prefix)"
+      jt16_link_name="$(arg jt16_link_name)"
+      jt16_xyz="$(arg jt16_xyz)"
+      jt16_rpy="$(arg jt16_rpy)"
       parent="$(arg prefix)base_link">
     <origin

Commit message: Update Hesai Lidar integration and documentation for SANEHAL-2

File: sanehal_vehicle_description/urdf/sanehal.urdf.xacro (robot description, xacro)
@@ -3,6 +3,8 @@
 <robot xmlns:xacro="http://www.ros.org/wiki/xacro" name="diffdrive_robot">
   <xacro:arg name="prefix" default="" />
-  <xacro:arg name="jt16_link_name" default="lidar_link" />
-  <xacro:arg name="jt16_xyz" default="0 0 0" />
+  <!-- Must match Hesai driver's ros.ros_frame_id (Issue #30). -->
+  <xacro:arg name="jt16_link_name" default="hesai_lidar" />
+  <!-- Measured from sanehal_base_link to the JT16 bottom-center datum. -->
+  <xacro:arg name="jt16_xyz" default="-0.080 0 0.250" />
   <xacro:arg name="jt16_rpy" default="0 0 0" />
   <xacro:include filename="$(find sanehal_vehicle_description)/urdf/sanehal.xacro" />

File: sanehal_vehicle_description/urdf/sanehal.xacro (robot description, xacro)
@@ -2,5 +2,5 @@
   <robot xmlns:xacro="http://www.ros.org/wiki/xacro">
     <!-- ロボットの表示を行う本体部分 -->
-    <xacro:macro name="sanehal" params="prefix parent jt16_link_name:=lidar_link jt16_xyz:='0 0 0' jt16_rpy:='0 0 0' *origin">
+    <xacro:macro name="sanehal" params="prefix parent jt16_link_name:=hesai_lidar jt16_xyz:='0 0 0' jt16_rpy:='0 0 0' *origin">
     <!-- Constants for robot dimensions -->
     <xacro:property name="PI" value="3.1415926535897931"/>
@@ -22,4 +22,7 @@
     <xacro:property name="caster_wheel_z_offset" value="0.0124" />
     <xacro:property name="caster_wheel_radius" value="0.0124" />
+    <xacro:property name="jt16_length" value="0.075" />
+    <xacro:property name="jt16_width" value="0.075" />
+    <xacro:property name="jt16_height" value="0.064" />
     <!-- Base Link -->
     <link name="${prefix}sanehal_base_link">
@@ -46,8 +49,25 @@
         </inertial>
     </link>
-    <!-- JT16 sensor frame.
-         Geometry is intentionally omitted until a vendor mesh or measured size is provided.
-         The frame exists so Issue #30 can reuse the same TF frame_id. -->
-    <link name="${prefix}${jt16_link_name}" />
+    <!-- JT16 driver/optical frame.
+         The mounting transform is measured from sanehal_base_link to the
+         bottom-center datum, with the connector facing rearward.
+         Simplified geometry is centered half the enclosure height above this
+         bottom-center datum.
+         Issue #30 must set Hesai ros.ros_frame_id to this link name. -->
+    <link name="${prefix}${jt16_link_name}">
+      <visual>
+        <origin xyz="0 0 ${jt16_height / 2.0}" rpy="0 0 0" />
+        <geometry>
+          <box size="${jt16_length} ${jt16_width} ${jt16_height}" />
+        </geometry>
+        <material name="black" />
+      </visual>
+      <collision>
+        <origin xyz="0 0 ${jt16_height / 2.0}" rpy="0 0 0" />
+        <geometry>
+          <box size="${jt16_length} ${jt16_width} ${jt16_height}" />
+        </geometry>
+      </collision>
+    </link>
     <joint name="${prefix}jt16_joint" type="fixed">
       <parent link="${prefix}sanehal_base_link" />

File: sanehal_vehicle_description/urdf/sanehal_display.urdf.xacro (robot description, xacro)
@@ -3,6 +3,8 @@
 <robot xmlns:xacro="http://www.ros.org/wiki/xacro" name="diffdrive_robot">
   <xacro:arg name="prefix" default="" />
-  <xacro:arg name="jt16_link_name" default="lidar_link" />
-  <xacro:arg name="jt16_xyz" default="0 0 0" />
+  <!-- Must match Hesai driver's ros.ros_frame_id (Issue #30). -->
+  <xacro:arg name="jt16_link_name" default="hesai_lidar" />
+  <!-- Measured from sanehal_base_link to the JT16 bottom-center datum. -->
+  <xacro:arg name="jt16_xyz" default="-0.080 0 0.250" />
   <xacro:arg name="jt16_rpy" default="0 0 0" />
   <!-- Import Rviz colors -->
