Commit message: SANEHAL-2 URDF update and sanehal naming migration for Issue #23

File: sanehal_vehicle_description/ros2_control/sanehal.ros2_control.xacro (robot description, xacro)
@@ -1,5 +1,5 @@
 <?xml version="1.0"?>
 <robot xmlns:xacro="http://www.ros.org/wiki/xacro">
-  <xacro:macro name="diffbot_ros2_control" params="name prefix">
+  <xacro:macro name="sanehal_ros2_control" params="name prefix">
     <ros2_control name="${name}" type="system">
       <hardware>

File: sanehal_vehicle_description/urdf/sanehal.urdf.xacro (robot description, xacro)
@@ -3,11 +3,11 @@
 <robot xmlns:xacro="http://www.ros.org/wiki/xacro" name="diffdrive_robot">
   <xacro:arg name="prefix" default="" />
-  <xacro:include filename="$(find sanehal_vehicle_description)/urdf/diffbot.xacro" />
+  <xacro:include filename="$(find sanehal_vehicle_description)/urdf/sanehal.xacro" />
   <!-- Import Rviz colors -->
-  <xacro:include filename="$(find sanehal_vehicle_description)/gazebo/diffbot.materials.xacro" />
-  <!-- Import diffbot ros2_control description -->
-  <xacro:include filename="$(find sanehal_vehicle_description)/ros2_control/diffbot.ros2_control.xacro" />
+  <xacro:include filename="$(find sanehal_vehicle_description)/gazebo/sanehal.materials.xacro" />
+  <!-- Import sanehal ros2_control description -->
+  <xacro:include filename="$(find sanehal_vehicle_description)/ros2_control/sanehal.ros2_control.xacro" />
   <link name="$(arg prefix)base_link" />
-  <xacro:diffbot
+  <xacro:sanehal
       prefix="$(arg prefix)"
       parent="$(arg prefix)base_link">
@@ -15,6 +15,6 @@
         xyz="0 0 0"
         rpy="0 0 0" />
-  </xacro:diffbot>
-  <xacro:diffbot_ros2_control
+  </xacro:sanehal>
+  <xacro:sanehal_ros2_control
     name="Sanehal" prefix="$(arg prefix)" />
 </robot>

File: sanehal_vehicle_description/urdf/sanehal.xacro (robot description, xacro)
@@ -2,19 +2,24 @@
   <robot xmlns:xacro="http://www.ros.org/wiki/xacro">
     <!-- ロボットの表示を行う本体部分 -->
-    <xacro:macro name="diffbot" params="prefix parent *origin">
+    <xacro:macro name="sanehal" params="prefix parent *origin">
     <!-- Constants for robot dimensions -->
     <xacro:property name="PI" value="3.1415926535897931"/>
     <xacro:property name="base_mass" value="2.0" /> <!-- arbitrary value for base mass -->
-    <xacro:property name="base_width" value="0.30750" /><!-- x -->
-    <xacro:property name="base_length" value="0.268" /><!-- y -->
-    <xacro:property name="base_height" value="0.45542" /> <!-- z -->
+    <xacro:property name="base_width" value="0.176" /><!-- x -->
+    <xacro:property name="base_length" value="0.175" /><!-- y -->
+    <xacro:property name="base_height" value="0.0545" /> <!-- z -->
+    <xacro:property name="base_x_offset" value="-0.03825" />
+    <xacro:property name="base_ground_clearance" value="0.035" />
     <xacro:property name="wheel_mass" value="0.100" /> <!-- arbitrary value for wheel mass -->
-    <xacro:property name="wheel_len" value="0.020" />
-    <xacro:property name="wheel_radius" value="0.03925" /> <!-- = 0.0785/2 -->
-    <xacro:property name="wheel_x_offset" value="0.12525" />
+    <xacro:property name="wheel_len" value="0.021" />
+    <xacro:property name="wheel_radius" value="0.0395" />
+    <xacro:property name="wheel_x_offset" value="0.0" />
+    <xacro:property name="wheel_y_offset" value="0.100" />
+    <xacro:property name="wheel_z_offset" value="0.035" />
     <xacro:property name="caster_wheel_mass" value="0.03" /> <!-- arbitrary value for caster wheel mass -->
-    <xacro:property name="caster_wheel_x_offset" value="-0.09175" /> <!-- arbitrary value for caster wheel mass -->
-    <xacro:property name="caster_wheel_radius" value="0.020" />
-    <xacro:property name="z_offset" value="-0" /> <!-- Space btw top of beam and the each joint -->
+    <xacro:property name="caster_wheel_x_offset" value="-0.09325" />
+    <xacro:property name="caster_wheel_y_offset" value="0.0" />
+    <xacro:property name="caster_wheel_z_offset" value="0.0124" />
+    <xacro:property name="caster_wheel_radius" value="0.0124" />
     <!-- add sensor file  -->
     <xacro:include filename="$(find ldlidar_stl_description)/urdf/ld19.xacro" />
@@ -22,5 +27,5 @@
     <link name="${prefix}sanehal_base_link">
       <collision>
-        <origin xyz="0 0 0" rpy="0 0 0"/>
+        <origin xyz="${base_x_offset} 0 ${base_ground_clearance + base_height/2}" rpy="0 0 0"/>
         <geometry>
           <box size="${base_width} ${base_length} ${base_height}"/>
@@ -28,5 +33,5 @@
       </collision>
       <visual>
-        <origin xyz="0 0 ${base_height/2}" rpy="0 0 0"/>
+        <origin xyz="${base_x_offset} 0 ${base_ground_clearance + base_height/2}" rpy="0 0 0"/>
         <geometry>
           <box size="${base_width} ${base_length} ${base_height}"/>
@@ -35,5 +40,5 @@
       </visual>
       <inertial>
-        <origin xyz="0 0 0" rpy="0 0 0"/>
+        <origin xyz="${base_x_offset} 0 ${base_ground_clearance + base_height/2}" rpy="0 0 0"/>
         <mass value="${base_mass}"/>
         <inertia
@@ -133,5 +138,5 @@
       <parent link="${prefix}sanehal_base_link"/>
       <child link="${prefix}left_wheel"/>
-      <origin xyz="${wheel_x_offset} ${base_width/2} ${z_offset}" rpy="0 0 0"/>
+      <origin xyz="${wheel_x_offset} ${wheel_y_offset} ${wheel_z_offset}" rpy="0 0 0"/>
       <axis xyz="0 1 0"/>
       <dynamics damping="0.2"/>
@@ -140,5 +145,5 @@
       <parent link="${prefix}sanehal_base_link"/>
       <child link="${prefix}right_wheel"/>
-      <origin xyz="${wheel_x_offset} -${base_width/2} ${z_offset}" rpy="0 0 ${PI}"/>
+      <origin xyz="${wheel_x_offset} -${wheel_y_offset} ${wheel_z_offset}" rpy="0 0 ${PI}"/>
       <axis xyz="0 1 0"/>
       <dynamics damping="0.2"/>
@@ -147,5 +152,5 @@
       <parent link="${prefix}sanehal_base_link"/>
       <child link="${prefix}caster_rear_wheel"/>
-      <origin xyz="${-base_width/2 + caster_wheel_radius} 0 ${z_offset}" rpy="0 0 0"/>
+      <origin xyz="${caster_wheel_x_offset} ${caster_wheel_y_offset} ${caster_wheel_z_offset}" rpy="0 0 0"/>
     </joint>
   </xacro:macro>

File: sanehal_vehicle_description/urdf/sanehal_display.urdf.xacro (robot description, xacro)
@@ -4,8 +4,8 @@
   <xacro:arg name="prefix" default="" />
   <!-- Import Rviz colors -->
-  <xacro:include filename="$(find sanehal_vehicle_description)/gazebo/diffbot.materials.xacro" />
-  <xacro:include filename="$(find sanehal_vehicle_description)/urdf/diffbot.xacro" />
+  <xacro:include filename="$(find sanehal_vehicle_description)/gazebo/sanehal.materials.xacro" />
+  <xacro:include filename="$(find sanehal_vehicle_description)/urdf/sanehal.xacro" />
   <link name="$(arg prefix)base_link" />
-  <xacro:diffbot
+  <xacro:sanehal
       prefix="$(arg prefix)"
       parent="$(arg prefix)base_link">
@@ -13,4 +13,4 @@
         xyz="0 0 0"
         rpy="0 0 0" />
-  </xacro:diffbot>
+  </xacro:sanehal>
 </robot>

Commit message: Integrate SANEHAL-2 Robot bringup

File: sanehal_vehicle_description/ros2_control/sanehal.ros2_control.xacro (robot description, xacro)
@@ -1,19 +1,26 @@
 <?xml version="1.0"?>
 <robot xmlns:xacro="http://www.ros.org/wiki/xacro">
-  <xacro:macro name="sanehal_ros2_control" params="name prefix">
+  <xacro:macro name="sanehal_ros2_control"
+      params="name prefix use_mock_hardware:=false dynamixel_port:=/dev/dxhub dynamixel_baud_rate:=1000000">
     <ros2_control name="${name}" type="system">
       <hardware>
-        <plugin>dynamixel_hardware_interface/DynamixelHardware</plugin>
-        <param name="port_name">/dev/dxhub</param>
-        <param name="baud_rate">1000000</param>
-        <param name="error_timeout_ms">500</param>
-        <!-- Appended to the dynamixel_hardware_interface package share path. -->
-        <param name="dynamixel_model_folder">/param/dxl_model</param>
-        <param name="number_of_joints">2</param>
-        <param name="number_of_transmissions">2</param>
-        <param name="disable_torque_at_init">true</param>
-        <!-- ID 2 is the left motor; ID 1 is the oppositely mounted right motor. -->
-        <param name="transmission_to_joint_matrix">1, 0, 0, -1</param>
-        <param name="joint_to_transmission_matrix">1, 0, 0, -1</param>
+        <xacro:if value="${use_mock_hardware}">
+          <plugin>mock_components/GenericSystem</plugin>
+          <param name="calculate_dynamics">false</param>
+        </xacro:if>
+        <xacro:unless value="${use_mock_hardware}">
+          <plugin>dynamixel_hardware_interface/DynamixelHardware</plugin>
+          <param name="port_name">${dynamixel_port}</param>
+          <param name="baud_rate">${dynamixel_baud_rate}</param>
+          <param name="error_timeout_ms">500</param>
+          <!-- Appended to the dynamixel_hardware_interface package share path. -->
+          <param name="dynamixel_model_folder">/param/dxl_model</param>
+          <param name="number_of_joints">2</param>
+          <param name="number_of_transmissions">2</param>
+          <param name="disable_torque_at_init">true</param>
+          <!-- ID 2 is left; ID 1 is the oppositely mounted right motor. -->
+          <param name="transmission_to_joint_matrix">1, 0, 0, -1</param>
+          <param name="joint_to_transmission_matrix">1, 0, 0, -1</param>
+        </xacro:unless>
       </hardware>
       <joint name="${prefix}left_wheel_joint">
@@ -27,5 +34,6 @@
         <state_interface name="velocity"/>
       </joint>
-      <gpio name="left_wheel_dxl">
+      <xacro:unless value="${use_mock_hardware}">
+        <gpio name="left_wheel_dxl">
         <param name="type">dxl</param>
         <param name="ID">2</param>
@@ -36,6 +44,6 @@
         <param name="Operating Mode">1</param>
         <param name="Return Delay Time">0</param>
-      </gpio>
-      <gpio name="right_wheel_dxl">
+        </gpio>
+        <gpio name="right_wheel_dxl">
         <param name="type">dxl</param>
         <param name="ID">1</param>
@@ -46,5 +54,6 @@
         <param name="Operating Mode">1</param>
         <param name="Return Delay Time">0</param>
-      </gpio>
+        </gpio>
+      </xacro:unless>
     </ros2_control>
   </xacro:macro>

File: sanehal_vehicle_description/urdf/sanehal.urdf.xacro (robot description, xacro)
@@ -3,4 +3,7 @@
 <robot xmlns:xacro="http://www.ros.org/wiki/xacro" name="diffdrive_robot">
   <xacro:arg name="prefix" default="" />
+  <xacro:arg name="use_mock_hardware" default="false" />
+  <xacro:arg name="dynamixel_port" default="/dev/dxhub" />
+  <xacro:arg name="dynamixel_baud_rate" default="1000000" />
   <!-- Must match Hesai driver's ros.ros_frame_id (Issue #30). -->
   <xacro:arg name="jt16_link_name" default="hesai_lidar" />
@@ -13,5 +16,11 @@
   <!-- Import sanehal ros2_control description -->
   <xacro:include filename="$(find sanehal_vehicle_description)/ros2_control/sanehal.ros2_control.xacro" />
+  <link name="$(arg prefix)base_footprint" />
   <link name="$(arg prefix)base_link" />
+  <joint name="$(arg prefix)base_footprint_joint" type="fixed">
+    <parent link="$(arg prefix)base_footprint" />
+    <child link="$(arg prefix)base_link" />
+    <origin xyz="0 0 0" rpy="0 0 0" />
+  </joint>
   <xacro:sanehal
       prefix="$(arg prefix)"
@@ -25,4 +34,8 @@
   </xacro:sanehal>
   <xacro:sanehal_ros2_control
-    name="Sanehal" prefix="$(arg prefix)" />
+    name="Sanehal"
+    prefix="$(arg prefix)"
+    use_mock_hardware="$(arg use_mock_hardware)"
+    dynamixel_port="$(arg dynamixel_port)"
+    dynamixel_baud_rate="$(arg dynamixel_baud_rate)" />
 </robot>

File: sanehal_vehicle_description/urdf/sanehal_display.urdf.xacro (robot description, xacro)
@@ -11,5 +11,11 @@
   <xacro:include filename="$(find sanehal_vehicle_description)/gazebo/sanehal.materials.xacro" />
   <xacro:include filename="$(find sanehal_vehicle_description)/urdf/sanehal.xacro" />
+  <link name="$(arg prefix)base_footprint" />
   <link name="$(arg prefix)base_link" />
+  <joint name="$(arg prefix)base_footprint_joint" type="fixed">
+    <parent link="$(arg prefix)base_footprint" />
+    <child link="$(arg prefix)base_link" />
+    <origin xyz="0 0 0" rpy="0 0 0" />
+  </joint>
   <xacro:sanehal
       prefix="$(arg prefix)"
